File: pcb_design/MouseMinder.kicad_pcb (KiCad board)
At the start: 2 copper layers, 25.5 x 40.7 mm, 14 parts, among them J3 Conn_02x04_Odd_Even, SW1 LCK-TA022H18-2WL, U1 PMS150C

Commit message: Rev 6.1 turned a resistor 90 degrees for rework, updated the silkscreen.
Parts:
- added G***: LOGO, 0art:amanda_mouseminder_logo, B.Cu at (-21.6, 0.38)
- moved G*** 1.55 mm to (-20.2, 16.7)
- moved R1 0.97 mm to (-12.5, 28.7), turned to 90 degrees
Routing:
- net PIEZO: track 34.4 -> 36.6 mm
Other:
- board text added: "Designed by a human."
- board text added: "Mouse By Amanda"
- board text added: "REV 6.1 OCT. 2026"
- board text removed: "REV 6 AUG. 2026"
